File: Hardware/$file549BD866.sch (KiCad schematic (older format))
At the start: 38 parts, among them K1 RELAYPTH, K2 RELAYPTH, P11 CONN_4, P12 CONN_8, P13 CONN_1

Commit message: Added final Files
Parts:
- gave numbers to parts that had none: 7
Changed lines of the file:
@@
 $EndComp
 $Comp
-L GND #PWR08
+L GND #PWR11
 U 1 1 549BDF28
 P 9850 5750
-F 0 "#PWR08" H 9850 5750 30  0001 C CNN
+F 0 "#PWR11" H 9850 5750 30  0001 C CNN
 F 1 "GND" H 9850 5680 30  0001 C CNN
 F 2 "" H 9850 5750 60  0001 C CNN
@@
 	3500 6300 3600 6300
 $Comp
-L GND #PWR09
+L GND #PWR8
 U 1 1 549C0995
 P 3900 5200
-F 0 "#PWR09" H 3900 5200 30  0001 C CNN
+F 0 "#PWR8" H 3900 5200 30  0001 C CNN
 F 1 "GND" H 3900 5130 30  0001 C CNN
 F 2 "" H 3900 5200 60  0001 C CNN
@@
 	3900 5150 3900 5200
 $Comp
-L GND #PWR010
+L GND #PWR9
 U 1 1 549C0A48
 P 3900 6550
-F 0 "#PWR010" H 3900 6550 30  0001 C CNN
+F 0 "#PWR9" H 3900 6550 30  0001 C CNN
 F 1 "GND" H 3900 6480 30  0001 C CNN
 F 2 "" H 3900 6550 60  0001 C CNN
@@
 $EndComp
 $Comp
-L GND #PWR011
+L GND #PWR10
 U 1 1 549C155C
 P 7150 5500
-F 0 "#PWR011" H 7150 5500 30  0001 C CNN
+F 0 "#PWR10" H 7150 5500 30  0001 C CNN
 F 1 "GND" H 7150 5430 30  0001 C CNN
 F 2 "" H 7150 5500 60  0001 C CNN
@@
 	2000 6300 2000 5650
 $Comp
-L BC849 Q?
+L BC849 Q3
 U 1 1 5584F951
 P 4750 2850
-F 0 "Q?" H 4750 2701 40  0000 R CNN
+F 0 "Q3" H 4750 2701 40  0000 R CNN
 F 1 "BC849" H 4750 3000 40  0000 R CNN
 F 2 "SOT-23" H 4650 2952 29  0000 C CNN
@@
 $EndComp
 $Comp
-L BC849 Q?
+L BC849 Q4
 U 1 1 5584FCA7
 P 6250 2850
-F 0 "Q?" H 6250 2701 40  0000 R CNN
+F 0 "Q4" H 6250 2701 40  0000 R CNN
 F 1 "BC849" H 6250 3000 40  0000 R CNN
 F 2 "SOT-23" H 6150 2952 29  0000 C CNN
@@
 $EndComp
 $Comp
-L BC849 Q?
+L BC849 Q6
 U 1 1 5584FD82
 P 7750 2850
-F 0 "Q?" H 7750 2701 40  0000 R CNN
+F 0 "Q6" H 7750 2701 40  0000 R CNN
 F 1 "BC849" H 7750 3000 40  0000 R CNN
 F 2 "SOT-23" H 7650 2952 29  0000 C CNN
@@
 $EndComp
 $Comp
-L BC849 Q?
+L BC849 Q7
 U 1 1 5584FE88
 P 9250 2850
-F 0 "Q?" H 9250 2701 40  0000 R CNN
+F 0 "Q7" H 9250 2701 40  0000 R CNN
 F 1 "BC849" H 9250 3000 40  0000 R CNN
 F 2 "SOT-23" H 9150 2952 29  0000 C CNN
@@
 $EndComp
 $Comp
-L BC849 Q?
+L BC849 Q1
 U 1 1 558500BD
 P 3800 4950
-F 0 "Q?" H 3800 4801 40  0000 R CNN
+F 0 "Q1" H 3800 4801 40  0000 R CNN
 F 1 "BC849" H 3800 5100 40  0000 R CNN
 F 2 "SOT-23" H 3700 5052 29  0000 C CNN
@@
 $EndComp
 $Comp
-L BC849 Q?
+L BC849 Q2
 U 1 1 558503B2
 P 3800 6300
-F 0 "Q?" H 3800 6151 40  0000 R CNN
+F 0 "Q2" H 3800 6151 40  0000 R CNN
 F 1 "BC849" H 3800 6450 40  0000 R CNN
 F 2 "SOT-23" H 3700 6402 29  0000 C CNN
@@
 $EndComp
 $Comp
-L BC849 Q?
+L BC849 Q5
 U 1 1 5585062F
 P 7050 5150
-F 0 "Q?" H 7050 5001 40  0000 R CNN
+F 0 "Q5" H 7050 5001 40  0000 R CNN
 F 1 "BC849" H 7050 5300 40  0000 R CNN
 F 2 "SOT-23" H 6950 5252 29  0000 C CNN
