File: Hardware/MCU_BaseBoard.sch (KiCad schematic (older format))
At the start: 46 parts, among them IC2 LM1117, J1 USB_2, K4 CONN_3, P1 CONN_01X04, P10 CONN_1, P14 CONN_01X10, P15 CONN_01X10, P16 CONN_01X10, P17 CONN_01X10, P18 CONN_01X10, P19 CONN_01X10, P2 CONN_01X10, P20 CONN_01X10, P25 CONN_01X04, P26 CONN_01X04, P27 CONN_01X04, P29 CONN_01X04, P3 CONN_01X04, P4 CONN_01X04, P5 CONN_01X04, P6 CONN_1, P7 CONN_1, P8 CONN_1, P9 CONN_1, SW1 INT1, SW18 INT0, SW19 INT1, SW20 SPST, SW21 INT1, U1 7805, U8 CP2102

Commit message: verified schematic and component placement
corrections written on schematic and layout
Other:
- note added: "Create a 40 pin component with the name Explore MCU Breakout \nand also a footprint for it.\nDo not put it as individucal connectors,\n people may find difficult to understand what these connectors are!"
- note added: "If this LED indicates LED Power connect it to VBUS, \ndon't leave stand alone\n"

Commit message: added new files
Parts:
- removed C6: 0.1uf, symbol C
- removed J1: USB_2, symbol USB_2
- removed P1: CONN_01X04, symbol CONN_01X04
- removed P14, P15, P16, P17, P18, P19, P2, P20: CONN_01X10, symbol CONN_01X10
- removed R11, R12: 10k, symbol R
- removed SW1, SW21: INT1, symbol SPST
- removed U8: CP2102, MODULE, symbol CP2102
- added P1: CONN_01X02, symbol CONN_01X02
- added P14, P2: CONN_01X20, symbol CONN_01X20
- added P30: CONN_01X07, symbol CONN_01X07
- added U5: 40PIN_Breakout, symbol 40PIN_Breakout
Connections:
- net +5V: now also P14.1 (P1), P30.3 (P3), U5.40
- net GND: now also P14.2 (P2), P30.1 (P1), U5.39
- net RST: now also P2.12 (P12), U5.12
- net RX: now also P2.1 (P1), P30.4 (P4), U5.1
- net S1: now also P1.1 (P1)
- net S2: now also P1.2 (P2)
- net TX: now also P2.2 (P2), P30.5 (P5), U5.2
- net at JP10.1: now also P30.7 (P7)
- new net: P2.10 (P10), U5.10
- new net: P2.11 (P11), U5.11
- new net: P2.13 (P13), U5.13
- new net: P2.14 (P14), U5.14
- new net: P2.15 (P15), U5.15
- new net: P2.16 (P16), U5.16
- new net: P2.17 (P17), U5.17
- new net: P2.18 (P18), U5.18
- new net: P2.19 (P19), U5.19
- new net: P2.20 (P20), U5.20
- new net: P14.20 (P20), U5.21
- new net: P14.19 (P19), U5.22
- new net: P14.18 (P18), U5.23
- new net: P14.17 (P17), U5.24
- new net: P14.16 (P16), U5.25
- new net: P14.15 (P15), U5.26
- new net: P14.14 (P14), U5.27
- new net: P14.13 (P13), U5.28
- new net: P14.12 (P12), U5.29
- new net: P2.3 (P3), U5.3
- new net: P14.11 (P11), U5.30
- new net: P14.10 (P10), U5.31
- new net: P14.9 (P9), U5.32
- new net: P14.8 (P8), U5.33
- new net: P14.7 (P7), U5.34
- new net: P14.6 (P6), U5.35
- new net: P14.5 (P5), U5.36
- new net: P14.4 (P4), U5.37
- new net: P14.3 (P3), U5.38
- new net: P2.4 (P4), U5.4
- new net: P2.5 (P5), U5.5
- new net: P2.6 (P6), U5.6
- new net: P2.7 (P7), U5.7
- new net: P2.8 (P8), U5.8
- new net: P2.9 (P9), U5.9
- no-connect marks 24 -> 7
Other:
- note added: "Add SPI LCD"
- moved on the sheet: C3, JP10

Commit message: Added final Files
Parts:
- removed D1: BRIDGE, symbol BRIDGE
- added P15, P16: CONN_1, symbol CONN_1
- C2: value 100uF, 25V -> 100uF,25V
Connections:
- net 9V/12V: now also SW20.2
- net GND: now also K4.2 (PM), K4.3 (P3)
- no-connect marks 7 -> 9
Other:
- moved on the sheet: K4, SW20
Changed lines of the file:
@@
 P 5050 5750
 F 0 "C2" H 5100 5850 50  0000 L CNN
-F 1 "100uF, 25V" H 4850 5650 50  0000 L CNN
+F 1 "100uF,25V" H 4850 5650 50  0000 L CNN
 F 2 "" H 5050 5750 60  0001 C CNN
 F 3 "" H 5050 5750 60  0001 C CNN
@@
 L SPST SW20
 U 1 1 555AF883
-P 2150 4500
-F 0 "SW20" H 2150 4600 70  0000 C CNN
-F 1 "SPST" H 2150 4400 70  0000 C CNN
-F 2 "" H 2150 4500 60  0001 C CNN
-F 3 "" H 2150 4500 60  0001 C CNN
-	1    2150 4500
+P 2900 5350
+F 0 "SW20" H 2900 5450 70  0000 C CNN
+F 1 "SPST" H 2900 5250 70  0000 C CNN
+F 2 "" H 2900 5350 60  0001 C CNN
+F 3 "" H 2900 5350 60  0001 C CNN
+	1    2900 5350
 	1    0    0    -1
 $EndComp
@@
 F 3 "" H 1250 1600 60  0001 C CNN
 	1    1250 1600
-	1    0    0    -1
-$EndComp
-$Comp
-L BRIDGE D1
-U 1 1 555AF8BA
-P 2900 5350
-F 0 "D1" H 2900 5400 70  0000 C CNN
-F 1 "BRIDGE" H 2900 5300 70  0000 C CNN
-F 2 "" H 2900 5350 60  0001 C CNN
-F 3 "" H 2900 5350 60  0001 C CNN
-	1    2900 5350
 	1    0    0    -1
 $EndComp
@@
 L CONN_3 K4
 U 1 1 555AF8E2
-P 850 5150
-F 0 "K4" V 800 5150 50  0000 C CNN
-F 1 "CONN_3" V 900 5150 40  0000 C CNN
-F 2 "" H 850 5150 60  0000 C CNN
-F 3 "" H 850 5150 60  0000 C CNN
-	1    850  5150
+P 1800 5750
+F 0 "K4" V 1750 5750 50  0000 C CNN
+F 1 "CONN_3" V 1850 5750 40  0000 C CNN
+F 2 "" H 1800 5750 60  0000 C CNN
+F 3 "" H 1800 5750 60  0000 C CNN
+	1    1800 5750
 	-1   0    0    -1
 $EndComp
@@
 RST
 Wire Wire Line
-	1250 4500 1250 5050
-Connection ~ 1250 5250
-Wire Wire Line
-	2000 6300 2000 5350
-Wire Wire Line
-	2000 5350 2050 5350
-Wire Wire Line
-	2900 6500 2900 6200
-Wire Wire Line
-	1250 6500 2900 6500
-Wire Wire Line
-	1250 5150 1250 6500
-Wire Wire Line
-	1250 5050 1200 5050
-Wire Wire Line
-	1250 5150 1200 5150
-Wire Wire Line
-	1200 5250 1250 5250
-Wire Wire Line
 	4650 6300 4650 5650
 Connection ~ 4650 6300
@@
 Wire Notes Line
 	2950 600  2950 4250
-Wire Wire Line
-	2650 4500 2900 4500
-Wire Wire Line
-	1650 4500 1250 4500
 Connection ~ 750  1600
 Wire Wire Line
@@
 Connection ~ 2350 1600
 Wire Wire Line
-	6000 6300 2000 6300
-Wire Wire Line
 	5050 6300 5050 5950
 Connection ~ 5050 6300
 Wire Wire Line
-	6000 5650 6000 6300
+	6000 6300 6000 5650
 Wire Wire Line
 	5500 5350 5700 5350
@@
 	6300 5400 6300 5350
 Wire Wire Line
-	3750 5350 4250 5350
+	3400 5350 4250 5350
 Wire Wire Line
 	4200 5550 4200 5350
@@
 Connection ~ 5300 950
 Connection ~ 5300 1050
+$Comp
+L CONN_1 P15
+U 1 1 55767A8E
+P 10300 1050
+F 0 "P15" H 10380 1050 40  0000 L CNN
+F 1 "CONN_1" H 10300 1105 30  0001 C CNN
+F 2 "" H 10300 1050 60  0000 C CNN
+F 3 "" H 10300 1050 60  0000 C CNN
+	1    10300 1050
+	1    0    0    -1
+$EndComp
+$Comp
+L CONN_1 P16
+U 1 1 55767BA5
+P 10300 1300
+F 0 "P16" H 10380 1300 40  0000 L CNN
+F 1 "CONN_1" H 10300 1355 30  0001 C CNN
+F 2 "" H 10300 1300 60  0000 C CNN
+F 3 "" H 10300 1300 60  0000 C CNN
+	1    10300 1300
+	1    0    0    -1
+$EndComp
+NoConn ~ 10150 1050
+NoConn ~ 10150 1300
+Wire Wire Line
+	2150 5650 2150 5350
+Wire Wire Line
+	2150 5350 2400 5350
+Wire Wire Line
+	2150 5750 2150 6300
+Wire Wire Line
+	2150 6300 6000 6300
+Connection ~ 2150 5850
 $EndSCHEMATC
